File: hardware/control/control.kicad_sch (KiCad schematic)
At the start: 5 parts, among them J1 Conn_01x02_Pin, J2 USB_C_Receptacle, J3 Conn_01x02_Pin, Q1 2N7002, U2 DRV8220DSG

Commit message: done routing
Parts:
- added R10, R12: 10k, Resistor_SMD:R_0603_1608Metric, symbol Device:R
- added R36: 100, Resistor_SMD:R_0603_1608Metric, symbol Device:R
Connections:
- net +3V3: now also R36.2; no longer J3.1 (Pin_1)
- net GND: now also R10.2, R12.1
- net at J2.A5 (CC1): now also R12.2
- net at J2.B5 (CC2): now also R10.1
- new net: J3.1 (Pin_1), R36.1
Other:
- moved on the sheet: J3
