File: hardware/control/power.kicad_sch (KiCad schematic)
At the start: 12 parts, among them SW3 KMS221GLFS, U5 STI3508, U7 NCP163AFCT330T2G

Commit message: done routing
Parts:
- removed C15, C16: 1u, Capacitor_SMD:C_0603_1608Metric, symbol Device:C
- removed U7: NCP163AFCT330T2G, Package_CSP:WLCSP-4_0.64x0.64mm_Layout2x2_P0.35mm, symbol Regulator_Linear:NCP163AFCT330T2G
- added D7: SS210, Diode_SMD:D_SMA, symbol Device:D
Connections:
- net +5V: now also C31.1, L3.1, SW3.2, U5.5 (V_in), D7.1 (K)
- removed net V_bat: BT2.1 (+), C31.1, L3.1, SW3.2, U5.5 (V_in)
- new net: BT2.1 (+), D7.2 (A)
Other:
- moved on the sheet: BT2, C31, C32, D5, L3, R11, R9, SW3, U5
