File: hardware/control/control.kicad_pcb (KiCad board)
At the start: 4 copper layers, 47 x 26 mm, 43 parts, among them J1 Conn_01x02_Pin, J2 USB_C_Receptacle, J3 Conn_01x02_Pin, J5 Conn_01x02_Pin, Q1 2N7002, Q2 2N7002, SW2 KMS221GLFS, SW3 KMS221GLFS, SW4 KMS221GLFS, SW5 KMS221GLFS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

Commit message: changed inductor for jlc compliance
Parts:
- removed L3: 22u, Inductor_SMD:L_Wuerth_MAPI-4030
- added L5: 22u, Inductor_SMD:L_Changjiang_FTC303020D, F.Cu at (137.9, 114.0)
- L4: footprint Inductor_SMD:L_Wuerth_MAPI-4030 -> Inductor_SMD:L_Changjiang_FTC303020D
- moved L4 0.68 mm to (122.4, 114.1)
Routing:
- net /+5V: track 49.0 -> 48.2 mm
